Commit message: adding camera

File: urdf/velodyne.husky.xacro (robot description, xacro)
@@ -1,4 +1,4 @@
 <?xml version="1.0"?>
-<robot xmlns:xacro="http://www.ros.org/wiki/xacro" name="velodyned_husky">
+<robot xmlns:xacro="http://www.ros.org/wiki/xacro" name="velodyne_husky">
   <xacro:arg name="gpu" default="false"/>
   <xacro:property name="gpu" value="$(arg gpu)" />
@@ -9,5 +9,5 @@
   <xacro:property name="velodyne_rpy" value="$(arg velodyne_rpy)" />
   <xacro:include filename="$(find velodyne_description)/urdf/VLP-16.urdf.xacro"/>
-  <material name="black">
+  <material name="velodyne_support_black">
     <color rgba="0 0 0 1"/>
   </material>
@@ -18,5 +18,5 @@
       </geometry>
       <origin rpy="0 0 0" xyz="0 0 0"/>
-      <material name="black"/>
+      <material name="velodyne_support_black"/>
     </visual>
     <collision>
