Commit message: turning according to cbd but not moving forward

File: urdf/camera.husky.xacro (robot description, xacro)
@@ -1,4 +1,5 @@
 <?xml version="1.0"?>
 <robot xmlns:xacro="http://www.ros.org/wiki/xacro" name="camera_husky">
+  <xacro:property name="M_PI" value="3.1415926535897931" />
   <xacro:arg name="camera_xyz" default="0.0 0.0 0.05" />
   <xacro:property name="camera_xyz" value="$(arg camera_xyz)" />
@@ -33,5 +34,5 @@
   </gazebo>
   <GenericCamera parent="camera_support">
-    <origin xyz="${camera_xyz}" rpy="${camera_rpy}" />
+    <origin xyz="${camera_xyz}" rpy="${camera_rpy}" fov="${M_PI/1.5}" />
   </GenericCamera>
 </robot>

File: urdf/velodyne.husky.xacro (robot description, xacro)
@@ -35,5 +35,5 @@
     <material>Gazebo/Black</material>
   </gazebo>
-  <VLP-16 parent="velodyne_support" name="velodyne" topic="/velodyne_points" hz="5" samples="2000" gpu="${gpu}" max_range="105">
+  <VLP-16 parent="velodyne_support" name="velodyne" topic="/velodyne_points" hz="10" samples="1000" gpu="${gpu}" max_range="105">
     <origin xyz="${velodyne_xyz}" rpy="${velodyne_rpy}" />
   </VLP-16>

Commit message: all right

File: urdf/camera.husky.xacro (robot description, xacro)
@@ -34,5 +34,5 @@
   </gazebo>
   <GenericCamera parent="camera_support">
-    <origin xyz="${camera_xyz}" rpy="${camera_rpy}" fov="${M_PI/1.5}" />
+    <origin xyz="${camera_xyz}" rpy="${camera_rpy}" fov="${M_PI/3}" />
   </GenericCamera>
 </robot>
